File: Power-plug-reveng.kicad_sch (KiCad schematic)
At the start: 54 parts, among them K1 SW_Push, Q1 NMOSFETSOT23

Commit message: commit of POC code
Parts:
- R2, R3: value 12M -> 1.2M
Changed lines of the file:
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@@
       (effects (font (size 1.27 1.27)) (justify right))
     )
-    (property "Value" "12M" (id 1) (at 41.91 76.2 0)
+    (property "Value" "1.2M" (id 1) (at 41.91 76.2 0)
       (effects (font (size 1.27 1.27)) (justify right))
     )
@@
       (effects (font (size 1.27 1.27)) (justify right))
     )
-    (property "Value" "12M" (id 1) (at 41.91 83.82 0)
+    (property "Value" "1.2M" (id 1) (at 41.91 83.82 0)
       (effects (font (size 1.27 1.27)) (justify right))
     )
@@
     )
     (path "/31586cd4-60ce-432c-acab-437680ac0516"
-      (reference "R2") (unit 1) (value "12M") (footprint "")
+      (reference "R2") (unit 1) (value "1.2M") (footprint "")
     )
     (path "/05b8257f-4837-40ff-83a9-aab2f51831f1"
-      (reference "R3") (unit 1) (value "12M") (footprint "")
+      (reference "R3") (unit 1) (value "1.2M") (footprint "")
     )
     (path "/471009a1-3e06-4fa3-b556-e3cfdb98a486"
